File: pcb/battery_charger.kicad_pcb (KiCad board)
At the start: 2 copper layers, 29 x 18.5 mm, 20 parts, among them J1 USB_B_Micro, U1 TP4056, U2 DW01A, U3 FS8205A

Commit message: Se realizan correcciones al PCB
Parts:
- added FID1: Fiducial, Fiducial:Fiducial_0.5mm_Mask1mm, F.Cu at (104.0, 120.8)
- renumbered + to J2, - to J3, OUT+ to J4, B+ to J5, B- to J6, OUT- to J7
Routing:
- net +5V: track 41.2 -> 42.3 mm
Other:
- board text added: "+"
- board text added: "Grilla componentes: 0.5mm - 0.25mm Grilla pistas: 0.25mm Vías: 1mm (Límite Mayer 8mils - 0.80mm) Agujeros: 0.5mm (Límite Mayer 8mils - 0.40mm) Pistas: 0.75mm - 0.5mm - 0.25mm (Límite Mayer 8mils - 0.20mm) Clearance: 0.3mm - 0.2mm para U3 (Límite Mayer 8mils - 0.18mm) FR4 - 1.6mm espesor Terminación HASL"
- board text removed: "Grilla componentes: 0.5mm - 0.25mm Grilla pistas: 0.25mm Vías: 1mm (Límite Mayer 8mils - 0.80mm) Pistas: 0.75mm - 0.5mm - 0.25mm (Límite Mayer 8mils - 0.20mm) Clearance: 0.3mm - 0.2mm para U3 (Límite Mayer 8mils - 0.18mm) FR4 - 1.6mm espesor Terminación HASL"
Changed lines of the file:
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@@
   (general
     (thickness 1.6)
-    (drawings 15)
+    (drawings 17)
     (tracks 108)
     (zones 0)
-    (modules 20)
+    (modules 21)
     (nets 20)
   )
@@
     (45 Margin user)
     (46 B.CrtYd user hide)
-    (47 F.CrtYd user)
+    (47 F.CrtYd user hide)
     (48 B.Fab user hide)
     (49 F.Fab user hide)
@@
     (add_net "Net-(U3-Pad8)")
   )
+  (module Fiducial:Fiducial_0.5mm_Mask1mm (layer F.Cu)
+    (at 104 120.75)
+    (descr "Circular Fiducial, 0.5mm bare copper, 1mm soldermask opening (Level C)")
+    (tags fiducial)
+    (attr smd)
+    (fp_text reference FID1 (at 0 0) (layer F.SilkS) hide
+      (effects (font (size 1 1) (thickness 0.15)))
+    )
+    (fp_text value Fiducial (at 0 1.5) (layer F.Fab)
+      (effects (font (size 1 1) (thickness 0.15)))
+    )
+    (fp_circle (center 0 0) (end 0.75 0) (layer F.CrtYd) (width 0.05))
+    (fp_text user %R (at 0 0) (layer F.Fab)
+      (effects (font (size 0.2 0.2) (thickness 0.04)))
+    )
+    (fp_circle (center 0 0) (end 0.5 0) (layer F.Fab) (width 0.1))
+    (pad "" smd circle (at 0 0) (size 0.5 0.5) (layers F.Cu F.Mask)
+      (solder_mask_margin 0.25) (clearance 0.25))
+  )
   (module Connector_Wire:SolderWirePad_1x01_Drill0.8mm (layer F.Cu)
     (at 129 123.25)
@@
     (tags connector)
     (attr virtual)
-    (fp_text reference OUT+ (at 0.25 -2.25) (layer F.SilkS)
+    (fp_text reference J4 (at 0.25 -2.25) (layer F.SilkS)
       (effects (font (size 0.7 0.7) (thickness 0.15)))
     )
@@
     (tags connector)
     (attr virtual)
-    (fp_text reference OUT- (at 0.25 -2) (layer F.SilkS)
+    (fp_text reference J7 (at 0.25 -2) (layer F.SilkS)
       (effects (font (size 0.7 0.7) (thickness 0.15)))
     )
@@
     (tags connector)
     (attr virtual)
-    (fp_text reference B- (at 0 -2) (layer F.SilkS)
+    (fp_text reference J6 (at 0 -2) (layer F.SilkS)
       (effects (font (size 0.7 0.7) (thickness 0.15)))
     )
@@
     (tags connector)
     (attr virtual)
-    (fp_text reference B+ (at 0 -2) (layer F.SilkS)
+    (fp_text reference J5 (at 0 -2) (layer F.SilkS)
       (effects (font (size 0.7 0.7) (thickness 0.15)))
     )
@@
     (tags connector)
     (attr virtual)
-    (fp_text reference - (at 2.25 0) (layer F.SilkS)
+    (fp_text reference J3 (at 2.25 0) (layer F.SilkS)
       (effects (font (size 1 1) (thickness 0.15)))
     )
@@
     (tags connector)
     (attr virtual)
-    (fp_text reference + (at 2.25 0) (layer F.SilkS)
+    (fp_text reference J2 (at 2.25 0) (layer F.SilkS)
       (effects (font (size 1 1) (thickness 0.15)))
     )
@@
     )
   )
+  (gr_text + (at 114.75 122.25) (layer F.SilkS)
+    (effects (font (size 0.75 0.75) (thickness 0.1875)))
+  )
+  (gr_text + (at 113.5 122.25) (layer F.SilkS)
+    (effects (font (size 0.75 0.75) (thickness 0.1875)))
+  )
   (gr_text 1 (at 121 128.75) (layer F.SilkS)
     (effects (font (size 0.5 0.5) (thickness 0.125)))
@@
     (effects (font (size 0.5 0.5) (thickness 0.125)))
   )
-  (gr_text "Grilla componentes: 0.5mm - 0.25mm\nGrilla pistas: 0.25mm\nVías: 1mm (Límite Mayer 8mils - 0.80mm)\nPistas: 0.75mm - 0.5mm - 0.25mm (Límite Mayer 8mils - 0.20mm)\nClearance: 0.3mm - 0.2mm para U3 (Límite Mayer 8mils - 0.18mm)\n\nFR4 - 1.6mm espesor\nTerminación HASL" (at 142.5 128.25) (layer Dwgs.User)
+  (gr_text "Grilla componentes: 0.5mm - 0.25mm\nGrilla pistas: 0.25mm\nVías: 1mm (Límite Mayer 8mils - 0.80mm)\nAgujeros: 0.5mm (Límite Mayer 8mils - 0.40mm)\nPistas: 0.75mm - 0.5mm - 0.25mm (Límite Mayer 8mils - 0.20mm)\nClearance: 0.3mm - 0.2mm para U3 (Límite Mayer 8mils - 0.18mm)\n\nFR4 - 1.6mm espesor\nTerminación HASL" (at 142.5 128.25) (layer Dwgs.User)
     (effects (font (size 1 1) (thickness 0.15)) (justify left))
   )
@@
     (arrow2b (pts (xy 102.5 115.5) (xy 103.626504 114.913579)))
   )
-  (gr_text "Rev. 1" (at 105.5 120.5) (layer F.SilkS)
+  (gr_text "Rev. 1" (at 106.75 120.5) (layer F.SilkS)
     (effects (font (size 0.7 0.7) (thickness 0.15)))
   )
@@
   (segment (start 107.75 120.5) (end 105.25 123) (width 0.75) (layer F.Cu) (net 1))
   (segment (start 105.25 123) (end 107.8 125.55) (width 0.75) (layer F.Cu) (net 1))
-  (segment (start 109.6075 128.2) (end 110.345 127.4625) (width 0.75) (layer F.Cu) (net 1))
+  (segment (start 109.6075 128.2) (end 110.345 127.4625) (width 0.5) (layer F.Cu) (net 1))
   (segment (start 112.1875 122.25) (end 112.1875 120.9375) (width 0.75) (layer F.Cu) (net 1))
   (segment (start 111.75 120.5) (end 107.75 120.5) (width 0.75) (layer F.Cu) (net 1))
   (segment (start 112.1875 120.9375) (end 111.75 120.5) (width 0.75) (layer F.Cu) (net 1))
-  (segment (start 112.1875 122.25) (end 116.0625 122.25) (width 0.75) (layer F.Cu) (net 1))
   (segment (start 116.0625 121.3125) (end 116.0625 122.25) (width 0.75) (layer F.Cu) (net 1))
   (segment (start 116 121.25) (end 116.0625 121.3125) (width 0.5) (layer F.Cu) (net 1))
@@
   (segment (start 107.8 125.55) (end 107.8 127.55) (width 0.75) (layer F.Cu) (net 1))
   (segment (start 108.45 128.2) (end 108.25 128) (width 0.5) (layer F.Cu) (net 1))
-  (segment (start 109.6075 128.2) (end 108.45 128.2) (width 0.75) (layer F.Cu) (net 1))
-  (segment (start 110.345 128.55) (end 110.345 127.4625) (width 0.75) (layer F.Cu) (net 1))
-  (segment (start 111.295 129.5) (end 110.345 128.55) (width 0.75) (layer F.Cu) (net 1))
+  (segment (start 109.6075 128.2) (end 108.45 128.2) (width 0.5) (layer F.Cu) (net 1))
+  (segment (start 110.345 128.55) (end 110.345 127.4625) (width 0.5) (layer F.Cu) (net 1))
+  (segment (start 111.295 129.5) (end 110.345 128.55) (width 0.5) (layer F.Cu) (net 1))
   (segment (start 114 129.5) (end 111.295 129.5) (width 0.75) (layer F.Cu) (net 1))
   (segment (start 114.55071 130.05071) (end 114 129.5) (width 0.75) (layer F.Cu) (net 1))
-  (segment (start 114.55071 132.14179) (end 114.55071 130.05071) (width 0.75) (layer F.Cu) (net 1))
-  (segment (start 114.155 132.5375) (end 114.55071 132.14179) (width 0.75) (layer F.Cu) (net 1))
+  (segment (start 114.55071 132.14179) (end 114.55071 130.05071) (width 0.5) (layer F.Cu) (net 1))
+  (segment (start 114.155 132.5375) (end 114.55071 132.14179) (width 0.5) (layer F.Cu) (net 1))
+  (segment (start 111.75 120.5) (end 116.75 120.5) (width 0.75) (layer F.Cu) (net 1))
   (segment (start 106.7 130.8) (end 107.235002 130.8) (width 0.25) (layer F.Cu) (net 2))
   (segment (start 106.28 131.22) (end 106.7 130.8) (width 0.25) (layer F.Cu) (net 2))
@@
   (segment (start 116 129.3075) (end 116 132.5) (width 0.5) (layer F.Cu) (net 5))
   (segment (start 114.155 127.4625) (end 116 129.3075) (width 0.5) (layer F.Cu) (net 5))
-  (segment (start 125.25 131) (end 129 127.25) (width 0.5) (layer B.Cu) (net 5))
-  (segment (start 117.5 131) (end 125.25 131) (width 0.5) (layer B.Cu) (net 5))
-  (segment (start 127.85 122.1) (end 129 123.25) (width 0.5) (layer F.Cu) (net 5))
-  (segment (start 126 122.1) (end 127.85 122.1) (width 0.5) (layer F.Cu) (net 5))
+  (segment (start 125.25 131) (end 129 127.25) (width 0.75) (layer B.Cu) (net 5))
+  (segment (start 117.5 131) (end 125.25 131) (width 0.75) (layer B.Cu) (net 5))
+  (segment (start 127.85 122.1) (end 129 123.25) (width 0.75) (layer F.Cu) (net 5))
+  (segment (start 126 122.1) (end 127.85 122.1) (width 0.75) (layer F.Cu) (net 5))
   (segment (start 129 127.25) (end 129 123.25) (width 0.75) (layer F.Cu) (net 5))
   (segment (start 119.0625 135.5625) (end 116 132.5) (width 0.5) (layer F.Cu) (net 5))
