File: pcb/battery_charger.sch (KiCad schematic (older format))
At the start: 20 parts, among them J1 USB_B_Micro, U1 TP4056, U2 DW01A, U3 FS8205A

Commit message: Primera version del PCB layout
Parts:
- removed H3: OUT+, MountingHole:MountingHole_3mm_Pad, symbol Mechanical:MountingHole_Pad
- removed H4: BAT+, MountingHole:MountingHole_3mm_Pad, symbol Mechanical:MountingHole_Pad
- removed H5: BAT-, MountingHole:MountingHole_3mm_Pad, symbol Mechanical:MountingHole_Pad
- removed H6: OUT-, MountingHole:MountingHole_3mm_Pad, symbol Mechanical:MountingHole_Pad
- added J4: OUT+, Connector_Wire:SolderWirePad_1x01_Drill1.2mm, symbol Connector_Generic:Conn_01x01
- added J5: BAT+, Connector_Wire:SolderWirePad_1x01_Drill1.2mm, symbol Connector_Generic:Conn_01x01
- added J6: BAT-, Connector_Wire:SolderWirePad_1x01_Drill1.2mm, symbol Connector_Generic:Conn_01x01
- added J7: OUT-, Connector_Wire:SolderWirePad_1x01_Drill1.2mm, symbol Connector_Generic:Conn_01x01
- C1, C2: footprint Capacitor_SMD:C_0603_1608Metric -> Capacitor_SMD:C_0805_2012Metric
- C3: footprint Capacitor_SMD:C_0603_1608Metric -> Capacitor_SMD:C_1206_3216Metric
- D1, D2: footprint LED_SMD:LED_0603_1608Metric -> LED_SMD:LED_0805_2012Metric
- J1: footprint Connector_USB:USB_Micro-B_Amphenol_10103594-0001LF_Horizontal -> Connector_USB:USB_Micro-B_Molex-105017-0001
- J2: renamed from H1; footprint MountingHole:MountingHole_3mm_Pad -> Connector_Wire:SolderWirePad_1x01_Drill1.2mm; symbol Mechanical:MountingHole_Pad -> Connector_Generic:Conn_01x01
- J3: renamed from H2; footprint MountingHole:MountingHole_3mm_Pad -> Connector_Wire:SolderWirePad_1x01_Drill1.2mm; symbol Mechanical:MountingHole_Pad -> Connector_Generic:Conn_01x01
- R1, R2, R3, R4, R5: footprint Resistor_SMD:R_0603_1608Metric -> Resistor_SMD:R_0805_2012Metric
Connections:
- net GND: now also J7.1 (Pin_1)
- net at C3.1, R5.2, U1.5 (BAT): now also J4.1 (Pin_1), J5.1 (Pin_1)
- net at C2.2, U2.6 (GND), U3.6 (S2)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: now also J6.1 (Pin_1)
Other:
- note added: "Up to 1A \ninput current"
Changed lines of the file:
@@
 F 0 "R2" V 3850 3400 50  0000 L CNN
 F 1 "1K" V 4050 3400 50  0000 L CNN
-F 2 "Resistor_SMD:R_0603_1608Metric" V 3880 3450 50  0001 C CNN
+F 2 "Resistor_SMD:R_0805_2012Metric" V 3880 3450 50  0001 C CNN
 F 3 "~" H 3950 3450 50  0001 C CNN
 	1    3950 3450
@@
 F 0 "R1" V 3850 3600 50  0000 L CNN
 F 1 "1K" V 3650 3600 50  0000 L CNN
-F 2 "Resistor_SMD:R_0603_1608Metric" V 3680 3650 50  0001 C CNN
+F 2 "Resistor_SMD:R_0805_2012Metric" V 3680 3650 50  0001 C CNN
 F 3 "~" H 3750 3650 50  0001 C CNN
 	1    3750 3650
@@
 F 0 "D1" H 3200 3550 50  0000 C CNN
 F 1 "LED-B" H 3200 3750 50  0000 C CNN
-F 2 "LED_SMD:LED_0603_1608Metric" H 3200 3650 50  0001 C CNN
+F 2 "LED_SMD:LED_0805_2012Metric" H 3200 3650 50  0001 C CNN
 F 3 "~" H 3200 3650 50  0001 C CNN
 	1    3200 3650
@@
 F 0 "D2" H 3500 3200 50  0000 C CNN
 F 1 "LED-R" H 3450 3300 50  0000 C CNN
-F 2 "LED_SMD:LED_0603_1608Metric" H 3500 3450 50  0001 C CNN
+F 2 "LED_SMD:LED_0805_2012Metric" H 3500 3450 50  0001 C CNN
 F 3 "~" H 3500 3450 50  0001 C CNN
 	1    3500 3450
@@
 F 0 "R3" V 5400 3400 50  0000 L CNN
 F 1 "1K" V 5200 3400 50  0000 L CNN
-F 2 "Resistor_SMD:R_0603_1608Metric" V 5230 3450 50  0001 C CNN
+F 2 "Resistor_SMD:R_0805_2012Metric" V 5230 3450 50  0001 C CNN
 F 3 "~" H 5300 3450 50  0001 C CNN
 	1    5300 3450
@@
 	1    0    0    -1
 $EndComp
-$Comp
-L Mechanical:MountingHole_Pad H1
-U 1 1 5D8D2026
-P 1150 3050
-F 0 "H1" V 1300 3150 50  0000 R CNN
-F 1 "IN+" V 1000 3150 50  0000 R CNN
-F 2 "MountingHole:MountingHole_3mm_Pad" H 1150 3050 50  0001 C CNN
-F 3 "~" H 1150 3050 50  0001 C CNN
-	1    1150 3050
-	0    -1   -1   0
-$EndComp
-Wire Wire Line
-	1250 3050 1700 3050
 Connection ~ 1700 3050
 $Comp
-L Mechanical:MountingHole_Pad H2
+L Connector_Generic:Conn_01x01 J3
 U 1 1 5D8D6FE3
-P 1150 4150
-F 0 "H2" V 1300 4250 50  0000 R CNN
-F 1 "IN-" V 1000 4250 50  0000 R CNN
-F 2 "MountingHole:MountingHole_3mm_Pad" H 1150 4150 50  0001 C CNN
-F 3 "~" H 1150 4150 50  0001 C CNN
-	1    1150 4150
-	0    -1   -1   0
+P 1050 4150
+F 0 "J3" H 1100 4050 50  0000 R CNN
+F 1 "IN-" H 1100 4250 50  0000 R CNN
+F 2 "Connector_Wire:SolderWirePad_1x01_Drill1.2mm" H 1050 4150 50  0001 C CNN
+F 3 "~" H 1050 4150 50  0001 C CNN
+	1    1050 4150
+	-1   0    0    1
 $EndComp
 Wire Wire Line
@@
 F 0 "C1" H 2750 3750 50  0000 L CNN
 F 1 "0.1uF" H 2750 3550 50  0000 L CNN
-F 2 "Capacitor_SMD:C_0603_1608Metric" H 2738 3500 50  0001 C CNN
+F 2 "Capacitor_SMD:C_0805_2012Metric" H 2738 3500 50  0001 C CNN
 F 3 "~" H 2700 3650 50  0001 C CNN
 	1    2700 3650
@@
 F 0 "J1" H 2250 4050 50  0000 R CNN
 F 1 "USB_B_Micro" H 2450 3950 50  0000 R CNN
-F 2 "Connector_USB:USB_Micro-B_Amphenol_10103594-0001LF_Horizontal" H 2350 3550 50  0001 C CNN
+F 2 "Connector_USB:USB_Micro-B_Molex-105017-0001" H 2350 3550 50  0001 C CNN
 F 3 "~" H 2350 3550 50  0001 C CNN
 	1    2200 3600
@@
 F 0 "R4" H 6250 3750 50  0000 L CNN
 F 1 "1K" H 6450 3750 50  0000 L CNN
-F 2 "Resistor_SMD:R_0603_1608Metric" V 6330 3750 50  0001 C CNN
+F 2 "Resistor_SMD:R_0805_2012Metric" V 6330 3750 50  0001 C CNN
 F 3 "~" H 6400 3750 50  0001 C CNN
 	1    6400 3750
 	1    0    0    -1
-$EndComp
-$Comp
-L Mechanical:MountingHole_Pad H3
-U 1 1 5D8C9BB7
-P 9750 2600
-F 0 "H3" V 9900 2700 50  0000 R CNN
-F 1 "OUT+" V 9600 2700 50  0000 R CNN
-F 2 "MountingHole:MountingHole_3mm_Pad" H 9750 2600 50  0001 C CNN
-F 3 "~" H 9750 2600 50  0001 C CNN
-	1    9750 2600
-	0    1    1    0
-$EndComp
-$Comp
-L Mechanical:MountingHole_Pad H4
-U 1 1 5D8CE5A6
-P 9750 3100
-F 0 "H4" V 9900 3200 50  0000 R CNN
-F 1 "BAT+" V 9600 3200 50  0000 R CNN
-F 2 "MountingHole:MountingHole_3mm_Pad" H 9750 3100 50  0001 C CNN
-F 3 "~" H 9750 3100 50  0001 C CNN
-	1    9750 3100
-	0    1    1    0
 $EndComp
 Wire Wire Line
@@
 F 0 "R5" V 8800 3050 50  0000 L CNN
 F 1 "0.1K" V 8600 3000 50  0000 L CNN
-F 2 "Resistor_SMD:R_0603_1608Metric" V 8630 3100 50  0001 C CNN
+F 2 "Resistor_SMD:R_0805_2012Metric" V 8630 3100 50  0001 C CNN
 F 3 "~" H 8700 3100 50  0001 C CNN
 	1    8700 3100
@@
 F 0 "C2" H 8300 3800 50  0000 L CNN
 F 1 "0.1uF" H 8300 3600 50  0000 L CNN
-F 2 "Capacitor_SMD:C_0603_1608Metric" H 8288 3550 50  0001 C CNN
+F 2 "Capacitor_SMD:C_0805_2012Metric" H 8288 3550 50  0001 C CNN
 F 3 "~" H 8250 3700 50  0001 C CNN
 	1    8250 3700
 	1    0    0    -1
 $EndComp
-$Comp
-L Mechanical:MountingHole_Pad H5
-U 1 1 5D8E04E5
-P 9750 4350
-F 0 "H5" V 9900 4450 50  0000 R CNN
-F 1 "BAT-" V 9600 4450 50  0000 R CNN
-F 2 "MountingHole:MountingHole_3mm_Pad" H 9750 4350 50  0001 C CNN
-F 3 "~" H 9750 4350 50  0001 C CNN
-	1    9750 4350
-	0    1    1    0
-$EndComp
 Wire Wire Line
 	7650 4350 8000 4350
@@
 	9100 2600 9100 3100
 Connection ~ 9100 2600
-Wire Wire Line
-	9100 2600 9650 2600
 Connection ~ 9100 3100
 Wire Wire Line
@@
 $EndComp
 $Comp
-L Mechanical:MountingHole_Pad H6
-U 1 1 5D90B8C3
-P 9750 4900
-F 0 "H6" V 9900 5000 50  0000 R CNN
-F 1 "OUT-" V 9600 5000 50  0000 R CNN
-F 2 "MountingHole:MountingHole_3mm_Pad" H 9750 4900 50  0001 C CNN
-F 3 "~" H 9750 4900 50  0001 C CNN
-	1    9750 4900
-	0    1    1    0
-$EndComp
-$Comp
 L power:GND #PWR06
 U 1 1 5D90D043
@@
 F 0 "C3" H 9150 3800 50  0000 L CNN
 F 1 "10uF" H 9150 3600 50  0000 L CNN
-F 2 "Capacitor_SMD:C_0603_1608Metric" H 9138 3550 50  0001 C CNN
+F 2 "Capacitor_SMD:C_1206_3216Metric" H 9138 3550 50  0001 C CNN
 F 3 "~" H 9100 3700 50  0001 C CNN
 	1    9100 3700
@@
 Wire Wire Line
 	9100 3850 9100 4050
+Wire Wire Line
+	1250 3050 1700 3050
+$Comp
+L Connector_Generic:Conn_01x01 J2
+U 1 1 5D8D2026
+P 1050 3050
+F 0 "J2" H 1100 2950 50  0000 R CNN
+F 1 "IN+" H 1100 3150 50  0000 R CNN
+F 2 "Connector_Wire:SolderWirePad_1x01_Drill1.2mm" H 1050 3050 50  0001 C CNN
+F 3 "~" H 1050 3050 50  0001 C CNN
+	1    1050 3050
+	-1   0    0    1
+$EndComp
+Text Notes 850  3700 0    50   ~ 0
+  Up to 1A \ninput current
+Wire Wire Line
+	9100 2600 9650 2600
+$Comp
+L Connector_Generic:Conn_01x01 J4
+U 1 1 5D991672
+P 9850 2600
+F 0 "J4" H 9900 2500 50  0000 R CNN
+F 1 "OUT+" H 10000 2700 50  0000 R CNN
+F 2 "Connector_Wire:SolderWirePad_1x01_Drill1.2mm" H 9850 2600 50  0001 C CNN
+F 3 "~" H 9850 2600 50  0001 C CNN
+	1    9850 2600
+	1    0    0    -1
+$EndComp
+$Comp
+L Connector_Generic:Conn_01x01 J5
+U 1 1 5D99E784
+P 9850 3100
+F 0 "J5" H 9900 3000 50  0000 R CNN
+F 1 "BAT+" H 10000 3200 50  0000 R CNN
+F 2 "Connector_Wire:SolderWirePad_1x01_Drill1.2mm" H 9850 3100 50  0001 C CNN
+F 3 "~" H 9850 3100 50  0001 C CNN
+	1    9850 3100
+	1    0    0    -1
+$EndComp
+$Comp
+L Connector_Generic:Conn_01x01 J6
+U 1 1 5D9A02C6
+P 9850 4350
+F 0 "J6" H 9900 4250 50  0000 R CNN
+F 1 "BAT-" H 10000 4450 50  0000 R CNN
+F 2 "Connector_Wire:SolderWirePad_1x01_Drill1.2mm" H 9850 4350 50  0001 C CNN
+F 3 "~" H 9850 4350 50  0001 C CNN
+	1    9850 4350
+	1    0    0    -1
+$EndComp
+$Comp
+L Connector_Generic:Conn_01x01 J7
+U 1 1 5D9A3497
+P 9850 4900
+F 0 "J7" H 9900 4800 50  0000 R CNN
+F 1 "OUT-" H 10000 5000 50  0000 R CNN
+F 2 "Connector_Wire:SolderWirePad_1x01_Drill1.2mm" H 9850 4900 50  0001 C CNN
+F 3 "~" H 9850 4900 50  0001 C CNN
+	1    9850 4900
+	1    0    0    -1
+$EndComp
 $EndSCHEMATC

Commit message: Se optimiza el area ocupada por el pcb
Parts:
- J1: footprint Connector_USB:USB_Micro-B_Molex-105017-0001 -> Connector_USB:USB_Micro-B_GCT_USB3076-30-A
Changed lines of the file:
@@
 F 0 "J1" H 2250 4050 50  0000 R CNN
 F 1 "USB_B_Micro" H 2450 3950 50  0000 R CNN
-F 2 "Connector_USB:USB_Micro-B_Molex-105017-0001" H 2350 3550 50  0001 C CNN
+F 2 "Connector_USB:USB_Micro-B_GCT_USB3076-30-A" H 2350 3550 50  0001 C CNN
 F 3 "~" H 2350 3550 50  0001 C CNN
 	1    2200 3600

Commit message: Correcciones a esquematico
Parts:
- C1, C2: Digikey # (none) -> 399-1169-2-ND
- C3: Digikey # (none) -> 399-8153-2-ND
- D1: Digikey # (none) -> 160-1645-2-ND
- D2: Digikey # (none) -> 160-1427-2-ND
- J1: Digikey # (none) -> 609-4616-1-ND
- J2, J3, J4, J5, J6, J7: footprint Connector_Wire:SolderWirePad_1x01_Drill1.2mm -> Connector_Wire:SolderWirePad_1x01_Drill0.8mm
- R1, R2, R3, R4: Digikey # (none) -> RPC0805JT1K00TR-ND
- R5: value 0.1K -> 100R; Digikey # (none) -> 2019-RK73B2ATTD101JTR-ND
- U1: Other Part # (none) -> Mouser: 453-DIO5158XS8
- U2: Other Part # (none) -> https://www.sunrom.com/p/dw01a-sot23-6-lithum-battery-prote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
- U3: Other Part # (none) -> https://www.sunrom.com/p/fs8205a-tssop-8
Connections:
- net GND: now also J1.6 (Shield)
- no-connect marks 7 -> 6
Other:
- note added: "Cargador de Batería"
- note added: "Corriente de entrada \n de hasta 1A"
- note added: "Precisión de carga: 1.5%\nTensión de plena carga: 4.2V"
- note added: "Protección de Batería"
- note added: "Tensión de entrada\n 4.5V-5.5V"
- note removed: "Battery Charger"
- note removed: "Battery Protection"
- note removed: "Up to 1A \ninput current"
Changed lines of the file:
@@
 encoding utf-8
 Sheet 1 1
-Title "Cargador de Batería con Protección - TP final DCI"
+Title "Réplica Cargador de Batería con Protección TP4056 - TP DCI"
 Date "2019-09-22"
-Rev "1"
+Rev "G. Gontad"
 Comp "Brignone Matías"
 Comment1 ""
@@
 F 2 "Package_SO:SOP-8_3.76x4.96mm_P1.27mm" H 4650 3750 50  0001 C CNN
 F 3 "" H 4650 3750 50  0001 C CNN
+F 4 "Mouser: 453-DIO5158XS8" H 4650 3350 50  0001 C CNN "Other Part #"
 	1    4650 3350
 	1    0    0    -1
@@
 F 2 "Resistor_SMD:R_0805_2012Metric" V 3880 3450 50  0001 C CNN
 F 3 "~" H 3950 3450 50  0001 C CNN
+F 4 "RPC0805JT1K00TR-ND" V 3950 3450 50  0001 C CNN "Digikey #"
 	1    3950 3450
 	0    1    1    0
@@
 F 2 "Resistor_SMD:R_0805_2012Metric" V 3680 3650 50  0001 C CNN
 F 3 "~" H 3750 3650 50  0001 C CNN
+F 4 "RPC0805JT1K00TR-ND" V 3750 3650 50  0001 C CNN "Digikey #"
 	1    3750 3650
 	0    -1   -1   0
@@
 F 2 "LED_SMD:LED_0805_2012Metric" H 3200 3650 50  0001 C CNN
 F 3 "~" H 3200 3650 50  0001 C CNN
+F 4 "160-1645-2-ND " H 3200 3650 50  0001 C CNN "Digikey #"
 	1    3200 3650
 	-1   0    0    1
@@
 F 2 "LED_SMD:LED_0805_2012Metric" H 3500 3450 50  0001 C CNN
 F 3 "~" H 3500 3450 50  0001 C CNN
+F 4 "160-1427-2-ND" H 3500 3450 50  0001 C CNN "Digikey #"
 	1    3500 3450
 	-1   0    0    1
@@
 F 2 "Resistor_SMD:R_0805_2012Metric" V 5230 3450 50  0001 C CNN
 F 3 "~" H 5300 3450 50  0001 C CNN
+F 4 "RPC0805JT1K00TR-ND" V 5300 3450 50  0001 C CNN "Digikey #"
 	1    5300 3450
 	0    -1   -1   0
@@
 F 0 "J3" H 1100 4050 50  0000 R CNN
 F 1 "IN-" H 1100 4250 50  0000 R CNN
-F 2 "Connector_Wire:SolderWirePad_1x01_Drill1.2mm" H 1050 4150 50  0001 C CNN
+F 2 "Connector_Wire:SolderWirePad_1x01_Drill0.8mm" H 1050 4150 50  0001 C CNN
 F 3 "~" H 1050 4150 50  0001 C CNN
 	1    1050 4150
@@
 F 2 "Capacitor_SMD:C_0805_2012Metric" H 2738 3500 50  0001 C CNN
 F 3 "~" H 2700 3650 50  0001 C CNN
+F 4 "399-1169-2-ND " H 2700 3650 50  0001 C CNN "Digikey #"
 	1    2700 3650
 	1    0    0    -1
@@
 F 2 "Connector_USB:USB_Micro-B_GCT_USB3076-30-A" H 2350 3550 50  0001 C CNN
 F 3 "~" H 2350 3550 50  0001 C CNN
+F 4 "609-4616-1-ND" H 2200 3600 50  0001 C CNN "Digikey #"
 	1    2200 3600
 	-1   0    0    -1
@@
 NoConn ~ 1900 3700
 NoConn ~ 1900 3800
-NoConn ~ 2300 4000
 $Comp
 L integrated_circuit_library:FS8205A U3
@@
 F 2 "Package_SO:TSSOP-8_4.4x3mm_P0.65mm" H 7300 4950 50  0001 C CNN
 F 3 "" H 7300 4950 50  0001 C CNN
+F 4 "https://www.sunrom.com/p/fs8205a-tssop-8" H 7300 4450 50  0001 C CNN "Other Part #"
 	1    7300 4450
 	1    0    0    -1
@@
 F 2 "Package_TO_SOT_SMD:SOT-23-6" H 7300 3650 50  0001 C CNN
 F 3 "" H 7300 3650 50  0001 C CNN
+F 4 "https://www.sunrom.com/p/dw01a-sot23-6-lithum-battery-protection-ic" H 7300 3300 50  0001 C CNN "Other Part #"
 	1    7300 3300
 	1    0    0    -1
@@
 F 2 "Resistor_SMD:R_0805_2012Metric" V 6330 3750 50  0001 C CNN
 F 3 "~" H 6400 3750 50  0001 C CNN
+F 4 "RPC0805JT1K00TR-ND" H 6400 3750 50  0001 C CNN "Digikey #"
 	1    6400 3750
 	1    0    0    -1
@@
 P 8700 3100
 F 0 "R5" V 8800 3050 50  0000 L CNN
-F 1 "0.1K" V 8600 3000 50  0000 L CNN
+F 1 "100R" V 8600 3000 50  0000 L CNN
 F 2 "Resistor_SMD:R_0805_2012Metric" V 8630 3100 50  0001 C CNN
 F 3 "~" H 8700 3100 50  0001 C CNN
+F 4 "2019-RK73B2ATTD101JTR-ND " H 8700 3100 50  0001 C CNN "Digikey #"
 	1    8700 3100
 	0    -1   -1   0
@@
 F 2 "Capacitor_SMD:C_0805_2012Metric" H 8288 3550 50  0001 C CNN
 F 3 "~" H 8250 3700 50  0001 C CNN
+F 4 "399-1169-2-ND " H 8250 3700 50  0001 C CNN "Digikey #"
 	1    8250 3700
 	1    0    0    -1
@@
 Wire Notes Line
 	1450 4850 1450 2350
-Text Notes 3150 2300 0    100  ~ 0
-Battery Charger
+Text Notes 3000 2300 0    100  ~ 0
+Cargador de Batería
 Wire Notes Line
 	6150 2350 9400 2350
@@
 	6150 5550 6150 2350
 Text Notes 7200 2300 0    100  ~ 0
-Battery Protection
+Protección de Batería
 $Comp
 L Device:C C3
@@
 F 2 "Capacitor_SMD:C_1206_3216Metric" H 9138 3550 50  0001 C CNN
 F 3 "~" H 9100 3700 50  0001 C CNN
+F 4 "399-8153-2-ND" H 9100 3700 50  0001 C CNN "Digikey #"
 	1    9100 3700
 	1    0    0    -1
@@
 F 0 "J2" H 1100 2950 50  0000 R CNN
 F 1 "IN+" H 1100 3150 50  0000 R CNN
-F 2 "Connector_Wire:SolderWirePad_1x01_Drill1.2mm" H 1050 3050 50  0001 C CNN
+F 2 "Connector_Wire:SolderWirePad_1x01_Drill0.8mm" H 1050 3050 50  0001 C CNN
 F 3 "~" H 1050 3050 50  0001 C CNN
 	1    1050 3050
 	-1   0    0    1
 $EndComp
-Text Notes 850  3700 0    50   ~ 0
-  Up to 1A \ninput current
+Text Notes 600  3500 0    50   ~ 0
+Corriente de entrada \n   de hasta 1A
 Wire Wire Line
 	9100 2600 9650 2600
@@
 F 0 "J4" H 9900 2500 50  0000 R CNN
 F 1 "OUT+" H 10000 2700 50  0000 R CNN
-F 2 "Connector_Wire:SolderWirePad_1x01_Drill1.2mm" H 9850 2600 50  0001 C CNN
+F 2 "Connector_Wire:SolderWirePad_1x01_Drill0.8mm" H 9850 2600 50  0001 C CNN
 F 3 "~" H 9850 2600 50  0001 C CNN
 	1    9850 2600
@@
 F 0 "J5" H 9900 3000 50  0000 R CNN
 F 1 "BAT+" H 10000 3200 50  0000 R CNN
-F 2 "Connector_Wire:SolderWirePad_1x01_Drill1.2mm" H 9850 3100 50  0001 C CNN
+F 2 "Connector_Wire:SolderWirePad_1x01_Drill0.8mm" H 9850 3100 50  0001 C CNN
 F 3 "~" H 9850 3100 50  0001 C CNN
 	1    9850 3100
@@
 F 0 "J6" H 9900 4250 50  0000 R CNN
 F 1 "BAT-" H 10000 4450 50  0000 R CNN
-F 2 "Connector_Wire:SolderWirePad_1x01_Drill1.2mm" H 9850 4350 50  0001 C CNN
+F 2 "Connector_Wire:SolderWirePad_1x01_Drill0.8mm" H 9850 4350 50  0001 C CNN
 F 3 "~" H 9850 4350 50  0001 C CNN
 	1    9850 4350
@@
 F 0 "J7" H 9900 4800 50  0000 R CNN
 F 1 "OUT-" H 10000 5000 50  0000 R CNN
-F 2 "Connector_Wire:SolderWirePad_1x01_Drill1.2mm" H 9850 4900 50  0001 C CNN
+F 2 "Connector_Wire:SolderWirePad_1x01_Drill0.8mm" H 9850 4900 50  0001 C CNN
 F 3 "~" H 9850 4900 50  0001 C CNN
 	1    9850 4900
 	1    0    0    -1
 $EndComp
+Wire Wire Line
+	2300 4000 2300 4150
+Wire Wire Line
+	2300 4150 2200 4150
+Text Notes 650  3800 0    50   ~ 0
+Tensión de entrada\n    4.5V-5.5V
+Text Notes 2850 5200 0    79   ~ 0
+Precisión de carga: 1.5%\nTensión de plena carga: 4.2V
 $EndSCHEMATC

Commit message: Se realizan correcciones al PCB
Parts:
- added FID1: Fiducial, Fiducial:Fiducial_0.5mm_Mask1mm, symbol Mechanical:Fiducial
Changed lines of the file:
@@
 Text Notes 2850 5200 0    79   ~ 0
 Precisión de carga: 1.5%\nTensión de plena carga: 4.2V
+$Comp
+L Mechanical:Fiducial FID1
+U 1 1 5DB52B46
+P 1750 5050
+F 0 "FID1" H 1835 5096 50  0000 L CNN
+F 1 "Fiducial" H 1835 5005 50  0000 L CNN
+F 2 "Fiducial:Fiducial_0.5mm_Mask1mm" H 1750 5050 50  0001 C CNN
+F 3 "~" H 1750 5050 50  0001 C CNN
+	1    1750 5050
+	1    0    0    -1
+$EndComp
 $EndSCHEMATC
